Commit message: GNC: refactor thruster_map to use URDF

File: simulation/navigator_gazebo/urdf/thruster.xacro (robot description, xacro)
@@ -63,4 +63,15 @@
       <dynamics friction="100" damping="0.3" />
     </joint>
+    <transmission name="${name}_thruster_transmission">
+      <type>transmission_interface/SimpleTransmission</type>
+      <actuator name="${name}_motor">
+        <!-- Linear Mapping from force to actuator "effort" (motor command) such that
+             -->
+        <mechanicalReduction>1.35</mechanicalReduction>
+      </actuator>
+      <joint name="${name}_engine_propeller_joint">
+        <hardwareInterface>hardware_interface/EffortJointInterface</hardwareInterface>
+      </joint>
+    </transmission>
   </xacro:macro>
 </robot>
