Commit message: SIMULATION: add update_rate param to depth sensor

File: simulation/mil_gazebo/xacro/depth.xacro (robot description, xacro)
@@ -1,5 +1,5 @@
 <?xml version="1.0"?>
 <robot xmlns:xacro="http://ros.org/wiki/xacro">
-  <xacro:macro name="mil_depth" params="name:=depth xyz:='0 0 0' rpy='0 0 0' rate:=100">
+  <xacro:macro name="mil_depth" params="name:=depth xyz:='0 0 0' rpy='0 0 0' rate:=20">
     <link name="${name}" />
     <joint name="${name}_joint" type="fixed">
@@ -12,4 +12,5 @@
         <frame_id>${name}</frame_id>
         <offset>${xyz} ${rpy}</offset>
+        <update_rate>${rate}</update_rate>
       </plugin>
     </gazebo>
