Commit message: SIMULATION: optionaly get drag/buoyancy from ros params

File: simulation/mil_gazebo/xacro/buoyancy.xacro (robot description, xacro)
@@ -2,9 +2,15 @@
 <robot xmlns:xacro="http://ros.org/wiki/xacro">
   <xacro:macro  name="mil_buoyancy"
-                params='volume'>
+                params='use_param:=False volume:=0.05 fluid_density:=1000 '>
     <plugin name="BuoyancyPlugin" filename="libmil_buoyancy_gazebo.so">
-      <fluid_density>1000</fluid_density>
+        <xacro:if value="${use_param}">
+          <volume_param>/robot_parameters/volume</volume_param>
+          <fluid_density_param>/robot_parameters/fluid_density</fluid_density_param>
+        </xacro:if>
+        <xacro:unless value="${use_param}">
+            <volume>${volume}</volume>
+            <fluid_density>1000</fluid_density>
+        </xacro:unless>
       <fluid_level>0.0</fluid_level>
-      <volume>${volume}</volume>
     </plugin>
   </xacro:macro>

File: simulation/mil_gazebo/xacro/drag.xacro (robot description, xacro)
@@ -1,9 +1,15 @@
 <?xml version="1.0"?>
 <robot xmlns:xacro="http://ros.org/wiki/xacro">
-  <xacro:macro name="mil_drag" params="linear_coeffs:='0 0 0' angular_coeffs:='0 0 0'">
+  <xacro:macro name="mil_drag" params="use_param:=False linear_coeffs:='0 0 0' angular_coeffs:='0 0 0'">
     <gazebo>
       <plugin filename="libmil_drag_gazebo.so" name="drag_plugin">
-        <linear_coeffs>${linear_coeffs}</linear_coeffs>
-        <angular_coeffs>${angular_coeffs}</angular_coeffs>
+        <xacro:if value="${use_param}">
+          <linear_coeffs_param>/robot_parameters/drag/linear_coeffs</linear_coeffs_param>
+          <angular_coeffs_param>/robot_parameters/drag/angular_coeffs</angular_coeffs_param>
+        </xacro:if>
+        <xacro:unless value="${use_param}">
+          <linear_coeffs>${linear_coeffs}</linear_coeffs>
+          <angular_coeffs>${angular_coeffs}</angular_coeffs>
+        </xacro:unless>
       </plugin>
     </gazebo>
