Commit message: INDYAV_GAZEBO: added p3d

File: IndyAV/simulation/indyav_gazebo/urdf/indyav_car.urdf.xacro (robot description, xacro)
@@ -3,4 +3,5 @@
   <xacro:include filename="$(find indyav_gazebo)/xacro/go_kart.xacro"/>
   <xacro:include filename="$(find indyav_gazebo)/xacro/wheels.xacro"/>
+  <xacro:include filename="$(find wamv_gazebo)/urdf/sensors/wamv_p3d.xacro"/>
   <link name="base_link">
     <xacro:body_inertial/>
@@ -12,4 +13,8 @@
     </collision>
   </link>
+  <!-- TODO: replace this with a sylphase img gps -->
+  <xacro:property name="namespace" value="indyav_car"/>
+  <xacro:property name="sensor_namespace" value="sensors"/>
+  <xacro:wamv_p3d/>
   <xacro:back_wheel name="back_left_wheel"  xyz="-1   0.4 -0.2"/>
   <xacro:back_wheel name="back_right_wheel"  xyz="-1 -0.4 -0.2"/>

Commit message: IndyAv: switched p3d to sylphase
fixed the sylphase task for indyav without copying the files from navigator

I created a rostest in python to demo the sylphase change. I commented out two of the property xacros in the urdf, removing them did nothing. I changed the doc files to show the sylphase change

I realied I did not commit all the changes. here are the rest

final commit: commented out p3d from roslaunch and fixed rostest

indyav: switched p3d to sylphase

prototype: made ins publish to enu

fixed method by which ins_odom is published to enu

added ins to base_link connection within tf.launch, adjusted location of ins tf to be inside car, fixed docs

cleaned up comments and bugs

attempted fix by adding tf depend

added tf import to test file

made minor change to be able to push again

File: IndyAV/simulation/indyav_gazebo/urdf/indyav_car.urdf.xacro (robot description, xacro)
@@ -3,5 +3,5 @@
   <xacro:include filename="$(find indyav_gazebo)/xacro/go_kart.xacro"/>
   <xacro:include filename="$(find indyav_gazebo)/xacro/wheels.xacro"/>
-  <xacro:include filename="$(find wamv_gazebo)/urdf/sensors/wamv_p3d.xacro"/>
+  <xacro:include filename="$(find navigator_gazebo)/urdf/sylphase.xacro" />
   <link name="base_link">
     <xacro:body_inertial/>
@@ -13,8 +13,6 @@
     </collision>
   </link>
-  <!-- TODO: replace this with a sylphase img gps -->
-  <xacro:property name="namespace" value="indyav_car"/>
-  <xacro:property name="sensor_namespace" value="sensors"/>
-  <xacro:wamv_p3d/>
+  <xacro:sylphase name="ins"
+                  xyz="0.05 0.0 0.05" rpy="0 0 0" />
   <xacro:back_wheel name="back_left_wheel"  xyz="-1   0.4 -0.2"/>
   <xacro:back_wheel name="back_right_wheel"  xyz="-1 -0.4 -0.2"/>

Commit message: added sylphase and fixed_link_persistent xacros to xacro folder as they are required to add sylphase to indyav urdf. deleted p3d xacro instance and include, and added the same sylphase instance as from the navigator urdf
fixed the sylphase task for indyav without copying the files from navigator

I created a rostest in python to demo the sylphase change. I commented out two of the property xacros in the urdf, removing them did nothing. I changed the doc files to show the sylphase change

I realied I did not commit all the changes. here are the rest

final commit: commented out p3d from roslaunch and fixed rostest

indyav: switched p3d to sylphase

File: IndyAV/simulation/indyav_gazebo/urdf/indyav_car.urdf.xacro (robot description, xacro)
@@ -3,5 +3,5 @@
   <xacro:include filename="$(find indyav_gazebo)/xacro/go_kart.xacro"/>
   <xacro:include filename="$(find indyav_gazebo)/xacro/wheels.xacro"/>
-  <xacro:include filename="$(find wamv_gazebo)/urdf/sensors/wamv_p3d.xacro"/>
+  <xacro:include filename="$(find navigator_gazebo)/urdf/sylphase.xacro" />
   <link name="base_link">
     <xacro:body_inertial/>
@@ -13,8 +13,8 @@
     </collision>
   </link>
-  <!-- TODO: replace this with a sylphase img gps -->
-  <xacro:property name="namespace" value="indyav_car"/>
-  <xacro:property name="sensor_namespace" value="sensors"/>
-  <xacro:wamv_p3d/>
+  <!-- <xacro:property name="namespace" value="indyav_car"/> -->
+  <!-- <xacro:property name="sensor_namespace" value="sensors"/> -->
+  <xacro:sylphase name="ins"
+                  xyz="0.579628 0.136525 1.392278" rpy="0 0 0" />
   <xacro:back_wheel name="back_left_wheel"  xyz="-1   0.4 -0.2"/>
   <xacro:back_wheel name="back_right_wheel"  xyz="-1 -0.4 -0.2"/>

Commit message: changing params for kart

File: IndyAV/simulation/indyav_gazebo/urdf/indyav_car.urdf.xacro (robot description, xacro)
@@ -14,7 +14,8 @@
   </link>
   <xacro:sylphase name="ins"
-                  xyz="0.05 0.0 0.05" rpy="0 0 0" />
-  <xacro:back_wheel name="back_left_wheel"  xyz="-1   0.4 -0.2"/>
-  <xacro:back_wheel name="back_right_wheel"  xyz="-1 -0.4 -0.2"/>
+                  xyz="-0.585 0.05 0" rpy="0 ${radians(0)} 0"/>
+  <!-- TODO: distance from base_link in all directions -->
+  <xacro:back_wheel name="back_left_wheel"   xyz="-1  0.6 -0.1"/>
+  <xacro:back_wheel name="back_right_wheel"  xyz="-1 -0.6 -0.1"/>
   <gazebo>
     <plugin name="back_wheel_plugin" filename="libbackwheel_plugin.so">
@@ -28,6 +29,6 @@
     </plugin>
   </gazebo>
-  <xacro:front_wheel name="front_left_wheel"  xyz="1 0.4 -0.2"/>
-  <xacro:front_wheel name="front_right_wheel"  xyz="1 -0.4 -0.2"/>
+  <xacro:front_wheel name="front_left_wheel"  xyz="1 0.6 -0.1"/>
+  <xacro:front_wheel name="front_right_wheel"  xyz="1 -0.6 -0.1"/>
   <gazebo>
     <plugin name="gazebo_ros_control" filename="libgazebo_ros_control.so"/>

File: IndyAV/simulation/indyav_gazebo/xacro/go_kart.xacro (robot description, xacro)
@@ -3,8 +3,9 @@
 <robot xmlns:xacro="http://ros.org/wiki/xacro" name="go_kart">
   <xacro:include filename="$(find mil_gazebo)/xacro/util.xacro"/>
-  <xacro:property name="chassis_length" value = "1.0"/> <!-- x -->
-  <xacro:property name="chassis_width" value = "0.75"/>  <!-- y -->
-  <xacro:property name="chassis_height" value = "0.25"/> <!-- z -->
-  <xacro:property name="chassis_mass" value = "50.0"/>
+  <!-- TODO distance from the steering point to steering point -->
+  <xacro:property name="chassis_length" value = "1.905"/> <!-- x -->
+  <xacro:property name="chassis_width"  value = "0.800"/> <!-- y -->
+  <xacro:property name="chassis_height" value = "0.4"/>  <!-- z -->
+  <xacro:property name="chassis_mass"   value = "67.950"/>
   <xacro:macro name="body_geometry">
     <geometry>

File: IndyAV/simulation/indyav_gazebo/xacro/wheels.xacro (robot description, xacro)
@@ -2,11 +2,13 @@
 <robot xmlns:xacro="http://ros.org/wiki/xacro" name="wheels">
   <xacro:include filename="$(find mil_gazebo)/xacro/util.xacro"/>
-  <xacro:property name="wheel_length" value="0.25"/>
-  <xacro:property name="wheel_width" value="0.25"/>
-  <xacro:property name="wheel_height" value="0.25"/>
-  <xacro:property name="wheel_mass" value="5"/>
-  <xacro:macro name="wheel_geometry">
+  <xacro:property name="back_wheel_radius" value="0.25"/>
+  <xacro:property name="back_wheel_width" value="0.25"/>
+  <xacro:property name="back_wheel_mass" value="2.25"/>
+  <xacro:property name="front_wheel_radius" value="0.25"/>
+  <xacro:property name="front_wheel_width" value="0.25"/>
+  <xacro:property name="front_wheel_mass" value="1.65"/>
+  <xacro:macro name="wheel_geometry" params="radius width">
     <geometry>
-      <box size="${wheel_length} ${wheel_width} ${wheel_height}"/>
+      <box size="${radius} ${width} ${radius}"/>
     </geometry>
   </xacro:macro>
@@ -29,20 +31,22 @@
     </gazebo>
   </xacro:macro>
-  <xacro:macro name="wheel_physical">
+  <xacro:macro name="wheel_physical" params="mass radius width">
     <inertial>
-      <mass value="${wheel_mass}"/>
-      <xacro:box_inertia x="${wheel_length}" y="${wheel_width}" z="${wheel_height}"
-                         mass="${wheel_mass}"/>
+      <mass value="${mass}"/>
+      <xacro:box_inertia x="${radius}" y="${width}" z="${radius}"
+                         mass="${mass}"/>
     </inertial>
     <collision>
-      <xacro:wheel_geometry/>
+      <xacro:wheel_geometry radius="${radius}" width="${width}"/>
     </collision>
     <visual>
-      <xacro:wheel_geometry/>
+      <xacro:wheel_geometry radius="${radius}" width="${width}"/>
     </visual>
   </xacro:macro>
   <xacro:macro name="back_wheel" params="name xyz parent_link:='base_link'">
     <link name="${name}_link">
-      <xacro:wheel_physical/>
+      <xacro:wheel_physical mass=  "${back_wheel_mass}"
+                            radius="${back_wheel_radius}"
+                            width= "${back_wheel_width}"/>
     </link>
     <joint name="${parent_link}_to_${name}_link_joint" type="fixed">
@@ -57,5 +61,7 @@
                                           max_deflection_right_deg:='30'">
     <link name="${name}_link">
-      <xacro:wheel_physical/>
+      <xacro:wheel_physical mass=  "${front_wheel_mass}"
+                            radius="${front_wheel_radius}"
+                            width= "${front_wheel_width}"/>
     </link>
     <joint name="${parent_link}_to_${name}_link_joint" type="revolute">

Commit message: INDYAV: Switched to rotating tires (and changes-to-vrx-gazebo-test)
created file to check if back wheels are touching ground, adjusted cart to move due to force from back tires, still some bugs to fix

fixed up indy model to where car moves due to torque of backwheels. Also, wheels are cylinders that rotate now.

attempted fix for flakey VRX test

fixed plugin formatting errors

included vrx changes

fixed VRX sandisland

completed requested changes: added back axle link, added friction comments, re-adjusted go_kart params, fixed documentation, put transmission in utils, checked if back_axle existed before using

fixed linting error

adjusted wheel velocity msg name, fixed orientation of the car as well

adjusted yaw, fixed duplicate xacro, made wheel origin xacros, moved INS tf

fixed documentation

changed vrx sandislandtest to allow for ten minutes

File: IndyAV/simulation/indyav_gazebo/urdf/indyav_car.urdf.xacro (robot description, xacro)
@@ -3,4 +3,5 @@
   <xacro:include filename="$(find indyav_gazebo)/xacro/go_kart.xacro"/>
   <xacro:include filename="$(find indyav_gazebo)/xacro/wheels.xacro"/>
+  <xacro:include filename="$(find indyav_gazebo)/xacro/axles.xacro"/>
   <xacro:include filename="$(find navigator_gazebo)/urdf/sylphase.xacro" />
   <link name="base_link">
@@ -13,21 +14,25 @@
     </collision>
   </link>
-  <xacro:sylphase name="ins"
-                  xyz="0.05 0.0 0.05" rpy="0 0 0" />
-  <xacro:back_wheel name="back_left_wheel"  xyz="-1   0.4 -0.2"/>
-  <xacro:back_wheel name="back_right_wheel"  xyz="-1 -0.4 -0.2"/>
+  <xacro:front_axle name="front_left_axle"  xyz="0.52 0.47 -0.2"/>
+  <xacro:front_axle name="front_right_axle"  xyz="0.52 -0.47 -0.2"/>
+  <xacro:front_wheel name="front_left_wheel" xyz="0 0 0" parent_link="front_left_axle_link"/>
+  <xacro:front_wheel name="front_right_wheel" xyz="0 0 0" parent_link="front_right_axle_link"/>
+  <xacro:back_axle name="back_axle" xyz="-0.52 0 -0.2"/>
+  <xacro:back_wheel name="back_left_wheel"  xyz="0 0.4825 0" parent_link="back_axle_link"/>
+  <xacro:back_wheel name="back_right_wheel"  xyz="0 -0.4825 0" parent_link="back_axle_link"/>
   <gazebo>
     <plugin name="back_wheel_plugin" filename="libbackwheel_plugin.so">
       <wheels>
-        <wheel_0> back_right_wheel_link </wheel_0>
-        <wheel_1> back_left_wheel_link </wheel_1>
+        <wheel_0> back_axle_link_to_back_right_wheel_link_joint </wheel_0>
+        <wheel_1> back_axle_link_to_back_left_wheel_link_joint </wheel_1>
       </wheels>
-      <max_thrust>1000</max_thrust>
+      <back_axle_joint> base_link_to_back_axle_link_joint </back_axle_joint>
+      <max_wheel_rotational_vel>1000</max_wheel_rotational_vel>
       <max_velocity>20</max_velocity>
       <topic_name> throttle </topic_name>
     </plugin>
   </gazebo>
-  <xacro:front_wheel name="front_left_wheel"  xyz="1 0.4 -0.2"/>
-  <xacro:front_wheel name="front_right_wheel"  xyz="1 -0.4 -0.2"/>
+  <xacro:sylphase name="ins"
+                  xyz="-0.585 0.0 0.0" rpy="0 0 0" />
   <gazebo>
     <plugin name="gazebo_ros_control" filename="libgazebo_ros_control.so"/>

File: IndyAV/simulation/indyav_gazebo/xacro/go_kart.xacro (robot description, xacro)
@@ -3,8 +3,8 @@
 <robot xmlns:xacro="http://ros.org/wiki/xacro" name="go_kart">
   <xacro:include filename="$(find mil_gazebo)/xacro/util.xacro"/>
-  <xacro:property name="chassis_length" value = "1.0"/> <!-- x -->
-  <xacro:property name="chassis_width" value = "0.75"/>  <!-- y -->
-  <xacro:property name="chassis_height" value = "0.25"/> <!-- z -->
-  <xacro:property name="chassis_mass" value = "50.0"/>
+  <xacro:property name="chassis_length" value = "1.89"/> <!-- x -->
+  <xacro:property name="chassis_width" value = "0.965"/>  <!-- y -->
+  <xacro:property name="chassis_height" value = "0.15"/> <!-- z -->
+  <xacro:property name="chassis_mass" value = "67.950"/>
   <xacro:macro name="body_geometry">
     <geometry>

File: IndyAV/simulation/indyav_gazebo/xacro/wheels.xacro (robot description, xacro)
@@ -2,47 +2,79 @@
 <robot xmlns:xacro="http://ros.org/wiki/xacro" name="wheels">
   <xacro:include filename="$(find mil_gazebo)/xacro/util.xacro"/>
-  <xacro:property name="wheel_length" value="0.25"/>
-  <xacro:property name="wheel_width" value="0.25"/>
-  <xacro:property name="wheel_height" value="0.25"/>
-  <xacro:property name="wheel_mass" value="5"/>
-  <xacro:macro name="wheel_geometry">
+  <xacro:property name="front_wheel_radius" value="0.127"/>
+  <xacro:property name="front_wheel_width" value="0.127"/>
+  <xacro:property name="front_wheel_mass" value="3"/>
+  <xacro:property name="back_wheel_radius" value="0.1335"/>
+  <xacro:property name="back_wheel_width" value="0.203"/>
+  <xacro:property name="back_wheel_mass" value="5"/>
+  <xacro:macro name="front_wheel_geometry">
     <geometry>
-      <box size="${wheel_length} ${wheel_width} ${wheel_height}"/>
+       <cylinder length="${front_wheel_width}" radius="${front_wheel_radius}"/>
     </geometry>
   </xacro:macro>
-  <xacro:macro name="wheel_surface">
-    <surface>
-      <friction>
-        <ode>
-          <mu>1000</mu> <!-- left / right  friction ,very high -->
-          <mu2>1</mu2> <!-- forwards / backwards friction, very low -->
-          <fdir1> 0 1 0 </fdir1>
-        </ode>
-      </friction>
-    </surface>
+  <xacro:macro name="back_wheel_geometry">
+    <geometry>
+       <cylinder length="${back_wheel_width}" radius="${back_wheel_radius}"/>
+    </geometry>
   </xacro:macro>
   <xacro:macro name="do_wheel_surface" params="name">
     <gazebo reference="${name}_link">
-      <collision>
-        <xacro:wheel_surface/>
-      </collision>
+      <mu1>500</mu1> <!-- friction parallel to the tire (wheels need friction to roll) -->
     </gazebo>
   </xacro:macro>
-  <xacro:macro name="wheel_physical">
+  <xacro:macro name="front_wheel_origin">
+     <origin rpy="0 1.5708 0"/>
+  </xacro:macro>
+  <xacro:macro name="back_wheel_origin">
+     <origin rpy="0 1.5708 1.5708"/>
+  </xacro:macro>
+  <xacro:macro name="front_wheel_physical">
     <inertial>
-      <mass value="${wheel_mass}"/>
-      <xacro:box_inertia x="${wheel_length}" y="${wheel_width}" z="${wheel_height}"
-                         mass="${wheel_mass}"/>
+      <xacro:front_wheel_origin/>
+      <mass value="${front_wheel_mass}"/>
+      <xacro:cylinder_inertia h="${front_wheel_width}" r="${front_wheel_radius}" mass="${front_wheel_mass}"/>
     </inertial>
     <collision>
-      <xacro:wheel_geometry/>
+      <xacro:front_wheel_origin/>
+      <xacro:front_wheel_geometry/>
     </collision>
     <visual>
-      <xacro:wheel_geometry/>
+      <xacro:front_wheel_origin/>
+      <xacro:front_wheel_geometry/>
     </visual>
   </xacro:macro>
+  <xacro:macro name="back_wheel_physical">
+    <inertial>
+      <xacro:back_wheel_origin/>
+      <mass value="${back_wheel_mass}"/>
+      <xacro:cylinder_inertia h="${back_wheel_width}" r="${back_wheel_radius}" mass="${back_wheel_mass}"/>
+    </inertial>
+    <collision>
+      <xacro:back_wheel_origin/>
+      <xacro:back_wheel_geometry/>
+    </collision>
+    <visual>
+      <xacro:back_wheel_origin/>
+      <xacro:back_wheel_geometry/>
+    </visual>
+  </xacro:macro>
+  <!--Front Wheel Xacro-->
+  <xacro:macro name="front_wheel" params="name xyz parent_link:='base_link'">
+    <link name="${name}_link">
+       <xacro:front_wheel_physical/>
+    </link>
+    <joint name="${parent_link}_to_${name}_link_joint" type="continuous">
+      <parent link="${parent_link}" />
+      <child link="${name}_link" />
+      <origin xyz="${xyz}" rpy="0 0 0"/>
+      <axis xyz="1 0 0"/>
+    </joint>
+    <xacro:do_wheel_surface name="${name}"/>
+    <xacro:joint_transmission name="${name}" parent_link="${parent_link}"/>
+  </xacro:macro>
+  <!--Back Wheel Xacro-->
   <xacro:macro name="back_wheel" params="name xyz parent_link:='base_link'">
     <link name="${name}_link">
-      <xacro:wheel_physical/>
+       <xacro:back_wheel_physical/>
     </link>
     <joint name="${parent_link}_to_${name}_link_joint" type="fixed">
@@ -53,29 +85,3 @@
     <xacro:do_wheel_surface name="${name}"/>
   </xacro:macro>
-  <xacro:macro name="front_wheel" params="name xyz parent_link:='base_link'
-                                          max_deflection_left_deg:='30'
-                                          max_deflection_right_deg:='30'">
-    <link name="${name}_link">
-      <xacro:wheel_physical/>
-    </link>
-    <joint name="${parent_link}_to_${name}_link_joint" type="revolute">
-      <parent link="${parent_link}" />
-      <child link="${name}_link" />
-      <limit lower="${radians(-1 * float(max_deflection_right_deg))}"
-             upper="${radians(float(max_deflection_left_deg))}" effort="10000" velocity="100"/>
-      <axis xyz="0 0 1"/>
-      <origin xyz="${xyz}" rpy="0 0 0"/>
-    </joint>
-    <xacro:do_wheel_surface name="${name}"/>
-    <transmission name="${name}_transmission">
-      <type>transmission_interface/SimpleTransmission</type>
-      <joint name="${parent_link}_to_${name}_link_joint">
-        <hardwareInterface>hardware_interface/EffortJointInterface</hardwareInterface>
-      </joint>
-      <actuator name="${name}_actuator">
-        <hardwareInterface>hardware_interface/EffortJointInterface</hardwareInterface>
-        <mechanicalReduction>1</mechanicalReduction>
-      </actuator>
-    </transmission>
-  </xacro:macro>
 </robot>

File: mil_common/simulation/mil_gazebo/xacro/util.xacro (robot description, xacro)
@@ -10,3 +10,23 @@
              izz="${((y*y) + (x*x))*mass/12.0}"/>
   </xacro:macro>
+  <xacro:macro name="cylinder_inertia" params="r h mass">
+    <inertia ixx="${((3*r*r) + (h*h))*mass/12.0}"
+             ixy="0.0"
+             ixz="0.0"
+             iyy="${((3*r*r) + (h*h))*mass/12.0}"
+             iyz="0.0"
+             izz="${(r*r)*mass/2.0}"/>
+  </xacro:macro>
+  <xacro:macro name="joint_transmission" params="name parent_link">
+    <transmission name="${name}_transmission">
+      <type>transmission_interface/SimpleTransmission</type>
+      <joint name="${parent_link}_to_${name}_link_joint">
+        <hardwareInterface>hardware_interface/EffortJointInterface</hardwareInterface>
+      </joint>
+      <actuator name="${name}_actuator">
+        <hardwareInterface>hardware_interface/EffortJointInterface</hardwareInterface>
+        <mechanicalReduction>1</mechanicalReduction>
+      </actuator>
+    </transmission>
+  </xacro:macro>
 </robot>
