Commit message: PR Changes 1

File: SubjuGator/simulation/sub8_gazebo/urdf/sub8.urdf.xacro (robot description, xacro)
@@ -39,5 +39,6 @@
                               lx="0.08825985" ly="0.08825985" lz="0.08825985" />
   <xacro:mil_dvl name="dvl" xyz="0.0908 0 -0.2459" rpy="0 0 0.785" gazebo_offset="0 0 -1" rate="6.5" />
-  <xacro:mil_inclinometer name="inclinometer" xyz="0 0 0" rpy="0 0 0" rate="210" lx="0.08825985" ly="0.08825985" lz="0.08825985" />
+  <!-- STIM300 Rate Options (Hz): 125, 250, 500, 1000, 2000 -->
+  <xacro:mil_inclinometer name="inclinometer" topic_name='/imu/inclinometer' queue_size='20' xyz="0.21236 0.00254 -0.10233" rpy="0 -1.571 0" rate="250" lx="0.08825985" ly="0.08825985" lz="0.08825985" />
   <xacro:mil_depth name="depth" xyz="-0.235 0 -0.170" rpy="0 0 0" rate="20" />
   <xacro:mil_passive_sonar name="hydrophones" xyz="-0.0908 0 -0.2459" rpy="0 0 1.571"

File: mil_common/simulation/mil_gazebo/xacro/inclinometer.xacro (robot description, xacro)
@@ -1,5 +1,6 @@
 <?xml version="1.0"?>
 <robot xmlns:xacro="http://ros.org/wiki/xacro">
-  <xacro:macro name="mil_inclinometer" params="name:=inclinometer parent:='base_link' xyz:='0 0 0' rpy='0 0 0' rate:=100 lx:=0 ly:=0 lz:=0">
+  <xacro:macro name="mil_inclinometer" params="name:=inclinometer parent:='base_link' topic_name:=/imu/inclinometer queue_size:=20
+                                               xyz:='0 0 0' rpy='0 0 0' rate:=100 lx:=0 ly:=0 lz:=0">
     <link name="${name}" />
     <joint name="${name}_joint" type="fixed">
@@ -21,4 +22,6 @@
         <plugin name="${name}_plugin" filename="libmil_inclinometer_gazebo.so">
           <frame_id>${name}</frame_id>
+          <topic>${topic_name}</topic>
+          <queue>${queue_size}</queue>
         </plugin>
       </sensor>
