Commit message: Add ROS and generic pre-commit hooks, also add to CI

File: SubjuGator/simulation/sub8_gazebo/urdf/sub8.urdf.xacro (robot description, xacro)
@@ -2,52 +2,61 @@
 <robot xmlns:xacro="http://ros.org/wiki/xacro" name="sub8">
   <!-- Include macros -->
-  <xacro:include filename="$(find mil_gazebo)/xacro/fixed_link.xacro" />
-  <xacro:include filename="$(find mil_gazebo)/xacro/camera.xacro" />
-  <xacro:include filename="$(find mil_gazebo)/xacro/buoyancy.xacro" />
-  <xacro:include filename="$(find mil_gazebo)/xacro/dvl.xacro" />
-  <xacro:include filename="$(find mil_gazebo)/xacro/imu_magnetometer.xacro" />
-  <xacro:include filename="$(find mil_gazebo)/xacro/depth.xacro" />
-  <xacro:include filename="$(find mil_gazebo)/xacro/drag.xacro" />
-  <xacro:include filename="$(find mil_gazebo)/xacro/passive_sonar.xacro" />
-  <xacro:include filename="$(find mil_gazebo)/xacro/inclinometer.xacro" />
+  <xacro:include filename="$(find mil_gazebo)/xacro/fixed_link.xacro"/>
+  <xacro:include filename="$(find mil_gazebo)/xacro/camera.xacro"/>
+  <xacro:include filename="$(find mil_gazebo)/xacro/buoyancy.xacro"/>
+  <xacro:include filename="$(find mil_gazebo)/xacro/dvl.xacro"/>
+  <xacro:include filename="$(find mil_gazebo)/xacro/imu_magnetometer.xacro"/>
+  <xacro:include filename="$(find mil_gazebo)/xacro/depth.xacro"/>
+  <xacro:include filename="$(find mil_gazebo)/xacro/drag.xacro"/>
+  <xacro:include filename="$(find mil_gazebo)/xacro/passive_sonar.xacro"/>
+  <xacro:include filename="$(find mil_gazebo)/xacro/inclinometer.xacro"/>
   <!-- Base link of sub -->
   <link name="base_link">
     <inertial>
       <!-- Mass from official weigh-in at RobotSub 2018 -->
-      <mass value="47.6" />
+      <mass value="47.6"/>
       <!-- Imported from old SDF model of Sub, unclear how these values were determined -->
-      <inertia ixx="1.18" ixy="-0.003" ixz="0.04" iyy="1.431" iyz="-0.034" izz="1.262" />
+      <inertia ixx="1.18" ixy="-0.003" ixz="0.04" iyy="1.431" iyz="-0.034" izz="1.262"/>
     </inertial>
     <visual name="visual">
       <geometry>
-        <mesh filename="package://sub8_missions/tools/sub8/sub_redux.dae" />
+        <mesh filename="package://sub8_missions/tools/sub8/sub_redux.dae"/>
       </geometry>
     </visual>
     <collision name="collision">
       <geometry>
-        <mesh filename="package://sub8_missions/tools/sub8/sub_redux.dae" />
+        <mesh filename="package://sub8_missions/tools/sub8/sub_redux.dae"/>
       </geometry>
     </collision>
   </link>
   <!-- Sensors -->
-  <xacro:mil_fixed_link name="front_stereo" parent="base_link" xyz="0.2559 0 0.1707" rpy="0 0 0" />
-  <xacro:mil_camera name="front_left_cam" parent="front_stereo" namespace="/camera/front/left" xyz="0 0.0445 0" rpy="0 0 0" />
-  <xacro:mil_camera name="front_right_cam" parent="front_stereo" namespace="/camera/front/right" xyz="0 -0.0445 0" rpy="0 0 0" />
-  <xacro:mil_camera name="down_left_cam" parent="base_link" namespace="/camera/down" xyz="0.054 0.105 -0.256" rpy="0 1.57 1.57" />
-  <xacro:mil_imu_magnetometer name="imu" parent="base_link" imu_topic='/imu/data_raw' xyz="0.21236 0.00254 -0.10233" rpy="0 -1.571 0" rate="210"
-                              ax="0.015707963" ay="0.015707963" az="0.015707963"
-                              lx="0.08825985" ly="0.08825985" lz="0.08825985" />
-  <xacro:mil_dvl name="dvl" xyz="0.0908 0 -0.2459" rpy="0 0 0.785" gazebo_offset="0 0 -1" rate="6.5" />
+  <xacro:mil_fixed_link name="front_stereo" parent="base_link" xyz="0.2559 0 0.1707" rpy="0 0 0"/>
+  <xacro:mil_camera name="front_left_cam" parent="front_stereo" namespace="/camera/front/left" xyz="0 0.0445 0" rpy="0 0 0"/>
+  <xacro:mil_camera name="front_right_cam" parent="front_stereo" namespace="/camera/front/right" xyz="0 -0.0445 0" rpy="0 0 0"/>
+  <xacro:mil_camera name="down_left_cam" parent="base_link" namespace="/camera/down" xyz="0.054 0.105 -0.256" rpy="0 1.57 1.57"/>
+  <xacro:mil_imu_magnetometer
+    name="imu"
+    parent="base_link"
+    imu_topic='/imu/data_raw'
+    xyz="0.21236 0.00254 -0.10233"
+    rpy="0 -1.571 0"
+    rate="210"
+    ax="0.015707963"
+    ay="0.015707963"
+    az="0.015707963"
+    lx="0.08825985"
+    ly="0.08825985"
+    lz="0.08825985"
+  />
+  <xacro:mil_dvl name="dvl" xyz="0.0908 0 -0.2459" rpy="0 0 0.785" gazebo_offset="0 0 -1" rate="6.5"/>
   <!-- STIM300 Rate Options (Hz): 125, 250, 500, 1000, 2000; Velocity Random Walk (vrw) and Correlation Time (ctime) taken from datasheet;
   Given same xyz/rpy as imu_magnetometer -->
-  <xacro:mil_inclinometer name="inclinometer" topic_name='/imu/inclinometer' queue_size='20' xyz="0.21236 0.00254 -0.10233" rpy="0 -1.571 0"
-			  rate="250" vrw="0.08" ctime="1" />
-  <xacro:mil_depth name="depth" xyz="-0.235 0 -0.170" rpy="0 0 0" rate="20" />
-  <xacro:mil_passive_sonar name="hydrophones" xyz="-0.0908 0 -0.2459" rpy="0 0 1.571"
-                           model="transdec_pinger" freq="37000" amplitude="1000"/>
+  <xacro:mil_inclinometer name="inclinometer" topic_name='/imu/inclinometer' queue_size='20' xyz="0.21236 0.00254 -0.10233" rpy="0 -1.571 0" rate="250" vrw="0.08" ctime="1"/>
+  <xacro:mil_depth name="depth" xyz="-0.235 0 -0.170" rpy="0 0 0" rate="20"/>
+  <xacro:mil_passive_sonar name="hydrophones" xyz="-0.0908 0 -0.2459" rpy="0 0 1.571" model="transdec_pinger" freq="37000" amplitude="1000"/>
   <!-- Other fixed frames -->
-  <xacro:mil_fixed_link name="blueview" parent="base_link" xyz="0.333 0 0.381" rpy="3.142 0 0" />
+  <xacro:mil_fixed_link name="blueview" parent="base_link" xyz="0.333 0 0.381" rpy="3.142 0 0"/>
   <!-- Dynamics simulation -->
-  <xacro:mil_drag use_param='True' />
+  <xacro:mil_drag use_param='True'/>
   <gazebo>
     <plugin name="sub8_thrusters" filename="libsub8_thrusters.so">
@@ -56,5 +65,5 @@
       <link>base_link</link>
     </plugin>
-    <xacro:mil_buoyancy use_param='True' />
+    <xacro:mil_buoyancy use_param='True'/>
   </gazebo>
   <!-- TODO: add blueview simulator using ray sensor -->

File: SubjuGator/simulation/sub8_gazebo/urdf/sub8_no_cams.urdf.xacro (robot description, xacro)
@@ -2,52 +2,61 @@
 <robot xmlns:xacro="http://ros.org/wiki/xacro" name="sub8">
   <!-- Include macros -->
-  <xacro:include filename="$(find mil_gazebo)/xacro/fixed_link.xacro" />
+  <xacro:include filename="$(find mil_gazebo)/xacro/fixed_link.xacro"/>
   <!-- <xacro:include filename="$(find mil_gazebo)/xacro/camera.xacro" /> -->
-  <xacro:include filename="$(find mil_gazebo)/xacro/buoyancy.xacro" />
-  <xacro:include filename="$(find mil_gazebo)/xacro/dvl.xacro" />
-  <xacro:include filename="$(find mil_gazebo)/xacro/imu_magnetometer.xacro" />
-  <xacro:include filename="$(find mil_gazebo)/xacro/depth.xacro" />
-  <xacro:include filename="$(find mil_gazebo)/xacro/drag.xacro" />
-  <xacro:include filename="$(find mil_gazebo)/xacro/passive_sonar.xacro" />
-  <xacro:include filename="$(find mil_gazebo)/xacro/inclinometer.xacro" />
+  <xacro:include filename="$(find mil_gazebo)/xacro/buoyancy.xacro"/>
+  <xacro:include filename="$(find mil_gazebo)/xacro/dvl.xacro"/>
+  <xacro:include filename="$(find mil_gazebo)/xacro/imu_magnetometer.xacro"/>
+  <xacro:include filename="$(find mil_gazebo)/xacro/depth.xacro"/>
+  <xacro:include filename="$(find mil_gazebo)/xacro/drag.xacro"/>
+  <xacro:include filename="$(find mil_gazebo)/xacro/passive_sonar.xacro"/>
+  <xacro:include filename="$(find mil_gazebo)/xacro/inclinometer.xacro"/>
   <!-- Base link of sub -->
   <link name="base_link">
     <inertial>
       <!-- Mass from official weigh-in at RobotSub 2018 -->
-      <mass value="47.6" />
+      <mass value="47.6"/>
       <!-- Imported from old SDF model of Sub, unclear how these values were determined -->
-      <inertia ixx="1.18" ixy="-0.003" ixz="0.04" iyy="1.431" iyz="-0.034" izz="1.262" />
+      <inertia ixx="1.18" ixy="-0.003" ixz="0.04" iyy="1.431" iyz="-0.034" izz="1.262"/>
     </inertial>
     <visual name="visual">
       <geometry>
-        <mesh filename="package://sub8_missions/tools/sub8/sub_redux.dae" />
+        <mesh filename="package://sub8_missions/tools/sub8/sub_redux.dae"/>
       </geometry>
     </visual>
     <collision name="collision">
       <geometry>
-        <mesh filename="package://sub8_missions/tools/sub8/sub_redux.dae" />
+        <mesh filename="package://sub8_missions/tools/sub8/sub_redux.dae"/>
       </geometry>
     </collision>
   </link>
   <!-- Sensors -->
-  <xacro:mil_fixed_link name="front_stereo" parent="base_link" xyz="0.2559 0 0.1707" rpy="0 0 0" />
+  <xacro:mil_fixed_link name="front_stereo" parent="base_link" xyz="0.2559 0 0.1707" rpy="0 0 0"/>
   <!-- <xacro:mil_camera name="front_left_cam" parent="front_stereo" namespace="/camera/front/left" xyz="0 0.0445 0" rpy="0 0 0" />
   <xacro:mil_camera name="front_right_cam" parent="front_stereo" namespace="/camera/front/right" xyz="0 -0.0445 0" rpy="0 0 0" />
   <xacro:mil_camera name="down_left_cam" parent="base_link" namespace="/camera/down" xyz="0.054 0.105 -0.256" rpy="0 1.57 1.57" /> -->
-  <xacro:mil_imu_magnetometer name="imu" parent="base_link" imu_topic='/imu/data_raw' xyz="0.21236 0.00254 -0.10233" rpy="0 -1.571 0" rate="210"
-                              ax="0.015707963" ay="0.015707963" az="0.015707963"
-                              lx="0.08825985" ly="0.08825985" lz="0.08825985" />
-  <xacro:mil_dvl name="dvl" xyz="0.0908 0 -0.2459" rpy="0 0 0.785" gazebo_offset="0 0 -1" rate="6.5" />
+  <xacro:mil_imu_magnetometer
+    name="imu"
+    parent="base_link"
+    imu_topic='/imu/data_raw'
+    xyz="0.21236 0.00254 -0.10233"
+    rpy="0 -1.571 0"
+    rate="210"
+    ax="0.015707963"
+    ay="0.015707963"
+    az="0.015707963"
+    lx="0.08825985"
+    ly="0.08825985"
+    lz="0.08825985"
+  />
+  <xacro:mil_dvl name="dvl" xyz="0.0908 0 -0.2459" rpy="0 0 0.785" gazebo_offset="0 0 -1" rate="6.5"/>
   <!-- STIM300 Rate Options (Hz): 125, 250, 500, 1000, 2000; Velocity Random Walk (vrw) and Correlation Time (ctime) taken from datasheet;
   Given same xyz/rpy as imu_magnetometer -->
-  <xacro:mil_inclinometer name="inclinometer" topic_name='/imu/inclinometer' queue_size='20' xyz="0.21236 0.00254 -0.10233" rpy="0 -1.571 0"
-			  rate="250" vrw="0.08" ctime="1" />
-  <xacro:mil_depth name="depth" xyz="-0.235 0 -0.170" rpy="0 0 0" rate="20" />
-  <xacro:mil_passive_sonar name="hydrophones" xyz="-0.0908 0 -0.2459" rpy="0 0 1.571"
-                           model="transdec_pinger" freq="37000" amplitude="1000"/>
+  <xacro:mil_inclinometer name="inclinometer" topic_name='/imu/inclinometer' queue_size='20' xyz="0.21236 0.00254 -0.10233" rpy="0 -1.571 0" rate="250" vrw="0.08" ctime="1"/>
+  <xacro:mil_depth name="depth" xyz="-0.235 0 -0.170" rpy="0 0 0" rate="20"/>
+  <xacro:mil_passive_sonar name="hydrophones" xyz="-0.0908 0 -0.2459" rpy="0 0 1.571" model="transdec_pinger" freq="37000" amplitude="1000"/>
   <!-- Other fixed frames -->
-  <xacro:mil_fixed_link name="blueview" parent="base_link" xyz="0.333 0 0.381" rpy="3.142 0 0" />
+  <xacro:mil_fixed_link name="blueview" parent="base_link" xyz="0.333 0 0.381" rpy="3.142 0 0"/>
   <!-- Dynamics simulation -->
-  <xacro:mil_drag use_param='True' />
+  <xacro:mil_drag use_param='True'/>
   <gazebo>
     <plugin name="sub8_thrusters" filename="libsub8_thrusters.so">
@@ -56,5 +65,5 @@
       <link>base_link</link>
     </plugin>
-    <xacro:mil_buoyancy use_param='True' />
+    <xacro:mil_buoyancy use_param='True'/>
   </gazebo>
   <!-- TODO: add blueview simulator using ray sensor -->

File: mil_common/simulation/mil_gazebo/xacro/buoyancy.xacro (robot description, xacro)
@@ -1,15 +1,14 @@
 <?xml version="1.0"?>
 <robot xmlns:xacro="http://ros.org/wiki/xacro">
-  <xacro:macro  name="mil_buoyancy"
-                params='use_param:=False volume:=0.05 fluid_density:=1000 '>
+  <xacro:macro name="mil_buoyancy" params='use_param:=False volume:=0.05 fluid_density:=1000 '>
     <plugin name="BuoyancyPlugin" filename="libmil_buoyancy_gazebo.so">
-        <xacro:if value="${use_param}">
-          <volume_param>/robot_parameters/volume</volume_param>
-          <fluid_density_param>/robot_parameters/fluid_density</fluid_density_param>
-        </xacro:if>
-        <xacro:unless value="${use_param}">
-            <volume>${volume}</volume>
-            <fluid_density>1000</fluid_density>
-        </xacro:unless>
+      <xacro:if value="${use_param}">
+        <volume_param>/robot_parameters/volume</volume_param>
+        <fluid_density_param>/robot_parameters/fluid_density</fluid_density_param>
+      </xacro:if>
+      <xacro:unless value="${use_param}">
+        <volume>${volume}</volume>
+        <fluid_density>1000</fluid_density>
+      </xacro:unless>
       <fluid_level>0.0</fluid_level>
     </plugin>

File: mil_common/simulation/mil_gazebo/xacro/camera.xacro (robot description, xacro)
@@ -2,19 +2,21 @@
 <robot xmlns:xacro="http://ros.org/wiki/xacro">
   <!-- Macro for inserting an engine with its propeller. -->
-  <xacro:macro  name="mil_camera"
-                params="name namespace:='/camera'
+  <xacro:macro
+    name="mil_camera"
+    params="name namespace:='/camera'
                         parent='base_link' xyz:='0 0 0' rpy:='0 0 0'
                         width:=960 height:=600 fov:=1.047 fps:=30
-                        k1:=0 k2:=0 t1:=0 t2:=0 k3:=0">
-    <link name="${name}" />
+                        k1:=0 k2:=0 t1:=0 t2:=0 k3:=0"
+  >
+    <link name="${name}"/>
     <joint name="${name}_to_${parent}" type="fixed">
-      <parent link="${parent}" />
-      <child link="${name}" />
-      <origin xyz="${xyz}" rpy="${rpy}" />
+      <parent link="${parent}"/>
+      <child link="${name}"/>
+      <origin xyz="${xyz}" rpy="${rpy}"/>
     </joint>
-    <link name="${name}_optical" />
+    <link name="${name}_optical"/>
     <joint name="${name}_to_${name}_optical" type="fixed">
-      <parent link="${name}" />
-      <child link="${name}_optical" />
+      <parent link="${name}"/>
+      <child link="${name}_optical"/>
       <origin xyz="0 0 0" rpy="${-pi/2} 0 ${-pi/2}"/>
     </joint>

File: mil_common/simulation/mil_gazebo/xacro/depth.xacro (robot description, xacro)
@@ -2,5 +2,5 @@
 <robot xmlns:xacro="http://ros.org/wiki/xacro">
   <xacro:macro name="mil_depth" params="name:=depth xyz:='0 0 0' rpy='0 0 0' rate:=20">
-    <link name="${name}" />
+    <link name="${name}"/>
     <joint name="${name}_joint" type="fixed">
       <origin xyz="${xyz}" rpy="${rpy}"/>

File: mil_common/simulation/mil_gazebo/xacro/dvl.xacro (robot description, xacro)
@@ -2,5 +2,5 @@
 <robot xmlns:xacro="http://ros.org/wiki/xacro">
   <xacro:macro name="mil_dvl" params="name:=dvl parent:='base_link' xyz:='0 0 0' rpy='0 0 0' gazebo_offset=:='0 0 0' rate:=1">
-    <link name="${name}" />
+    <link name="${name}"/>
     <joint name="${name}_joint" type="fixed">
       <origin xyz="${xyz}" rpy="${rpy}"/>

File: mil_common/simulation/mil_gazebo/xacro/fixed_link.xacro (robot description, xacro)
@@ -1,12 +1,11 @@
 <?xml version="1.0"?>
 <robot xmlns:xacro="http://ros.org/wiki/xacro">
-  <xacro:macro  name="mil_fixed_link"
-                params="name parent='base_link'
+  <xacro:macro name="mil_fixed_link" params="name parent='base_link'
                         xyz:='0 0 0' rpy:='0 0 0'">
-    <link name="${name}" />
+    <link name="${name}"/>
     <joint name="${name}_to_${parent}" type="fixed">
-      <parent link="${parent}" />
-      <child link="${name}" />
-      <origin xyz="${xyz}" rpy="${rpy}" />
+      <parent link="${parent}"/>
+      <child link="${name}"/>
+      <origin xyz="${xyz}" rpy="${rpy}"/>
     </joint>
   </xacro:macro>

File: mil_common/simulation/mil_gazebo/xacro/imu.xacro (robot description, xacro)
@@ -3,5 +3,5 @@
   <xacro:macro name="mil_imu" params="name:=imu parent:='base_link' topic:='/imu/data' xyz:='0 0 0' rpy='0 0 0' rate:=100
                                       ax:=0 ay:=0 az:=0 lx:=0 ly:=0 lz:=0">
-    <link name="${name}" />
+    <link name="${name}"/>
     <joint name="${name}_joint" type="fixed">
       <origin xyz="${xyz}" rpy="${rpy}"/>
@@ -15,12 +15,36 @@
         <imu>
           <linear_acceleration>
-            <x><noise type="gaussian"><stddev>${lx}</stddev></noise></x>
-            <y><noise type="gaussian"><stddev>${ly}</stddev></noise></y>
-            <z><noise type="gaussian"><stddev>${lz}</stddev></noise></z>
+            <x>
+              <noise type="gaussian">
+                <stddev>${lx}</stddev>
+              </noise>
+            </x>
+            <y>
+              <noise type="gaussian">
+                <stddev>${ly}</stddev>
+              </noise>
+            </y>
+            <z>
+              <noise type="gaussian">
+                <stddev>${lz}</stddev>
+              </noise>
+            </z>
           </linear_acceleration>
           <angular_velocity>
-            <x><noise type="gaussian"><stddev>${ax}</stddev></noise></x>
-            <y><noise type="gaussian"><stddev>${ay}</stddev></noise></y>
-            <z><noise type="gaussian"><stddev>${az}</stddev></noise></z>
+            <x>
+              <noise type="gaussian">
+                <stddev>${ax}</stddev>
+              </noise>
+            </x>
+            <y>
+              <noise type="gaussian">
+                <stddev>${ay}</stddev>
+              </noise>
+            </y>
+            <z>
+              <noise type="gaussian">
+                <stddev>${az}</stddev>
+              </noise>
+            </z>
           </angular_velocity>
         </imu>

File: mil_common/simulation/mil_gazebo/xacro/imu_magnetometer.xacro (robot description, xacro)
@@ -1,7 +1,10 @@
 <?xml version="1.0"?>
 <robot xmlns:xacro="http://ros.org/wiki/xacro">
-  <xacro:macro name="mil_imu_magnetometer" params="name:=imu parent:='base_link' imu_topic:='/imu/data_raw' xyz:='0 0 0' rpy='0 0 0' rate:=100
-                                                   ax:=0 ay:=0 az:=0 lx:=0 ly:=0 lz:=0">
-    <link name="${name}" />
+  <xacro:macro
+    name="mil_imu_magnetometer"
+    params="name:=imu parent:='base_link' imu_topic:='/imu/data_raw' xyz:='0 0 0' rpy='0 0 0' rate:=100
+                                                   ax:=0 ay:=0 az:=0 lx:=0 ly:=0 lz:=0"
+  >
+    <link name="${name}"/>
     <joint name="${name}_joint" type="fixed">
       <origin xyz="${xyz}" rpy="${rpy}"/>
@@ -15,12 +18,36 @@
         <imu>
           <linear_acceleration>
-            <x><noise type="gaussian"><stddev>${lx}</stddev></noise></x>
-            <y><noise type="gaussian"><stddev>${ly}</stddev></noise></y>
-            <z><noise type="gaussian"><stddev>${lz}</stddev></noise></z>
+            <x>
+              <noise type="gaussian">
+                <stddev>${lx}</stddev>
+              </noise>
+            </x>
+            <y>
+              <noise type="gaussian">
+                <stddev>${ly}</stddev>
+              </noise>
+            </y>
+            <z>
+              <noise type="gaussian">
+                <stddev>${lz}</stddev>
+              </noise>
+            </z>
           </linear_acceleration>
           <angular_velocity>
-            <x><noise type="gaussian"><stddev>${ax}</stddev></noise></x>
-            <y><noise type="gaussian"><stddev>${ay}</stddev></noise></y>
-            <z><noise type="gaussian"><stddev>${az}</stddev></noise></z>
+            <x>
+              <noise type="gaussian">
+                <stddev>${ax}</stddev>
+              </noise>
+            </x>
+            <y>
+              <noise type="gaussian">
+                <stddev>${ay}</stddev>
+              </noise>
+            </y>
+            <z>
+              <noise type="gaussian">
+                <stddev>${az}</stddev>
+              </noise>
+            </z>
           </angular_velocity>
         </imu>

File: mil_common/simulation/mil_gazebo/xacro/inclinometer.xacro (robot description, xacro)
@@ -1,7 +1,10 @@
 <?xml version="1.0"?>
 <robot xmlns:xacro="http://ros.org/wiki/xacro">
-  <xacro:macro name="mil_inclinometer" params="name:=inclinometer parent:='base_link' topic_name:=/imu/inclinometer queue_size:=20
-                                               xyz:='0 0 0' rpy='0 0 0' rate:=100 vrw:=0 ctime:=1">
-    <link name="${name}" />
+  <xacro:macro
+    name="mil_inclinometer"
+    params="name:=inclinometer parent:='base_link' topic_name:=/imu/inclinometer queue_size:=20
+                                               xyz:='0 0 0' rpy='0 0 0' rate:=100 vrw:=0 ctime:=1"
+  >
+    <link name="${name}"/>
     <joint name="${name}_joint" type="fixed">
       <origin xyz="${xyz}" rpy="${rpy}"/>

File: mil_common/simulation/mil_gazebo/xacro/magnetometer.xacro (robot description, xacro)
@@ -2,5 +2,5 @@
 <robot xmlns:xacro="http://ros.org/wiki/xacro">
   <xacro:macro name="mil_magnetometer" params="name:=magnetometer parent:='base_link' topic:='/imu/data' xyz:='0 0 0' rpy='0 0 0' rate:=100">
-    <link name="${name}" />
+    <link name="${name}"/>
     <joint name="${name}_joint" type="fixed">
       <origin xyz="${xyz}" rpy="${rpy}"/>

File: mil_common/simulation/mil_gazebo/xacro/passive_sonar.xacro (robot description, xacro)
@@ -11,5 +11,5 @@
       </plugin>
     </gazebo>
-    <link name="${name}" />
+    <link name="${name}"/>
     <joint name="${name}_joint" type="fixed">
       <origin xyz="${xyz}" rpy="${rpy}"/>

File: mil_common/simulation/mil_gazebo/xacro/util.xacro (robot description, xacro)
@@ -3,18 +3,8 @@
   <!-- determined by https://en.wikipedia.org/wiki/List_of_moments_of_inertia -->
   <xacro:macro name="box_inertia" params="x y z mass">
-    <inertia ixx="${((y*y) + (z*z))*mass/12.0}"
-             ixy="0.0"
-             ixz="0.0"
-             iyy="${((x*x) + (z*z))*mass/12.0}"
-             iyz="0.0"
-             izz="${((y*y) + (x*x))*mass/12.0}"/>
+    <inertia ixx="${((y*y) + (z*z))*mass/12.0}" ixy="0.0" ixz="0.0" iyy="${((x*x) + (z*z))*mass/12.0}" iyz="0.0" izz="${((y*y) + (x*x))*mass/12.0}"/>
   </xacro:macro>
   <xacro:macro name="cylinder_inertia" params="r h mass">
-    <inertia ixx="${((3*r*r) + (h*h))*mass/12.0}"
-             ixy="0.0"
-             ixz="0.0"
-             iyy="${((3*r*r) + (h*h))*mass/12.0}"
-             iyz="0.0"
-             izz="${(r*r)*mass/2.0}"/>
+    <inertia ixx="${((3*r*r) + (h*h))*mass/12.0}" ixy="0.0" ixz="0.0" iyy="${((3*r*r) + (h*h))*mass/12.0}" iyz="0.0" izz="${(r*r)*mass/2.0}"/>
   </xacro:macro>
   <xacro:macro name="joint_transmission" params="name parent_link">
