Commit message: made inertia same as sub8 as temporary solution to allowing sub9 to work in simulation

File: SubjuGator/simulation/sub8_gazebo/urdf/sub9.urdf.xacro (robot description, xacro)
@@ -16,6 +16,6 @@
       <!-- Mass from official weigh-in at RobotSub 2018 -->
       <!-- determined from solid works as of 2020-08-09-->
-      <mass value="21.5" />
-      <inertia ixx="0.4674" ixy="-0.003" ixz="0.02" iyy="0.983" iyz="-0.0003" izz="1.197" />
+      <mass value="47.6" />
+      <inertia ixx="1.18" ixy="-0.003" ixz="0.04" iyy="1.431" iyz="-0.034" izz="1.262" />
     </inertial>
     <visual name="visual">

Commit message: Fix sub9 movement by updating intertia values to match sub8

File: SubjuGator/simulation/sub8_gazebo/urdf/sub9.urdf.xacro (robot description, xacro)
@@ -16,6 +16,6 @@
       <!-- Mass from official weigh-in at RobotSub 2018 -->
       <!-- determined from solid works as of 2020-08-09-->
-      <mass value="21.5"/>
-      <inertia ixx="0.4674" ixy="-0.003" ixz="0.02" iyy="0.983" iyz="-0.0003" izz="1.197"/>
+      <mass value="47.6"/>
+      <inertia ixx="1.18" ixy="-0.003" ixz="0.04" iyy="1.431" iyz="-0.034" izz="1.262"/>
     </inertial>
     <visual name="visual">

Commit message: Update sub9 inertial values based on rectangular prism inertial tensor formula

File: SubjuGator/simulation/sub8_gazebo/urdf/sub9.urdf.xacro (robot description, xacro)
@@ -14,8 +14,9 @@
   <link name="base_link">
     <inertial>
-      <!-- Mass from official weigh-in at RobotSub 2018 -->
-      <!-- determined from solid works as of 2020-08-09-->
-      <mass value="47.6"/>
-      <inertia ixx="1.18" ixy="-0.003" ixz="0.04" iyy="1.431" iyz="-0.034" izz="1.262"/>
+      <!-- Rough estimate of RoboSub 2022 -->
+      <mass value="21.5"/>
+      <!-- Estimate of inertial tensor based on inertial tensor for rectangular prism -->
+      <!-- https://en.wikipedia.org/wiki/List_of_moments_of_inertia#List_of_3D_inertia_tensors -->
+      <inertia ixx="0.96105" ixy="0.003" ixz="-0.02" iyy="1.799" iyz="0.0003" izz="2.1286"/>
     </inertial>
     <visual name="visual">
