Commit message: Add CI improvements for Noetic (#764)
This PR adds a series of steps for CI beginning with ROS Noetic. These steps include:

* Adding a `pre-commit` config file with a series of linters

* Add CI steps based on each commit hash and checkout

* Build docs for each hash and publish as an artifact

* Run the static type checker `pyright` and the linter `pylint`

* Run `catkin_make` tests for each hash

File: NaviGator/simulation/navigator_gazebo/urdf/camera.xacro (robot description, xacro)
@@ -2,19 +2,21 @@
 <robot xmlns:xacro="http://ros.org/wiki/xacro">
   <!-- Macro for inserting an engine with its propeller. -->
-  <xacro:macro  name="navigator_camera"
-                params="name namespace:='/camera'
+  <xacro:macro
+    name="navigator_camera"
+    params="name namespace:='/camera'
                         parent='base_link' xyz:='0 0 0' rpy:='0 0 0'
                         width:=960 height:=600 fov:=1.047 fps:=30
-                        k1:=0 k2:=0 t1:=0 t2:=0 k3:=0">
-    <link name="${name}" />
+                        k1:=0 k2:=0 t1:=0 t2:=0 k3:=0"
+  >
+    <link name="${name}"/>
     <joint name="${name}_to_${parent}" type="fixed">
-      <parent link="${parent}" />
-      <child link="${name}" />
-      <origin xyz="${xyz}" rpy="${rpy}" />
+      <parent link="${parent}"/>
+      <child link="${name}"/>
+      <origin xyz="${xyz}" rpy="${rpy}"/>
     </joint>
-    <link name="${name}_optical" />
+    <link name="${name}_optical"/>
     <joint name="${name}_to_${name}_optical" type="fixed">
-      <parent link="${name}" />
-      <child link="${name}_optical" />
+      <parent link="${name}"/>
+      <child link="${name}_optical"/>
       <origin xyz="0 0 0" rpy="${-pi/2} 0 ${-pi/2}"/>
     </joint>

File: NaviGator/simulation/navigator_gazebo/urdf/fixed_link.xacro (robot description, xacro)
@@ -1,12 +1,11 @@
 <?xml version="1.0"?>
 <robot xmlns:xacro="http://ros.org/wiki/xacro">
-  <xacro:macro  name="fixed_link"
-                params="name parent='base_link'
+  <xacro:macro name="fixed_link" params="name parent='base_link'
                         xyz:='0 0 0' rpy:='0 0 0'">
-    <link name="${name}" />
+    <link name="${name}"/>
     <joint name="${name}_to_${parent}" type="fixed">
-      <parent link="${parent}" />
-      <child link="${name}" />
-      <origin xyz="${xyz}" rpy="${rpy}" />
+      <parent link="${parent}"/>
+      <child link="${name}"/>
+      <origin xyz="${xyz}" rpy="${rpy}"/>
     </joint>
   </xacro:macro>

File: NaviGator/simulation/navigator_gazebo/urdf/fixed_link_persistent.xacro (robot description, xacro)
@@ -1,9 +1,8 @@
 <?xml version="1.0"?>
 <robot xmlns:xacro="http://ros.org/wiki/xacro">
-  <xacro:macro  name="fixed_link_persistent"
-                params="name parent='base_link'
+  <xacro:macro name="fixed_link_persistent" params="name parent='base_link'
                         xyz:='0 0 0' rpy:='0 0 0'">
     <gazebo>
-      <link name="${name}" />
+      <link name="${name}"/>
       <joint name="${name}_to_${parent}" type="fixed">
         <parent>${parent}</parent>
@@ -12,9 +11,9 @@
       </joint>
     </gazebo>
-    <link name="${name}" />
+    <link name="${name}"/>
     <joint name="${name}_to_${parent}" type="fixed">
-      <parent link="${parent}" />
-      <child link="${name}" />
-      <origin xyz="${xyz}" rpy="${rpy}" />
+      <parent link="${parent}"/>
+      <child link="${name}"/>
+      <origin xyz="${xyz}" rpy="${rpy}"/>
     </joint>
   </xacro:macro>

File: NaviGator/simulation/navigator_gazebo/urdf/navigator.urdf.xacro (robot description, xacro)
@@ -2,39 +2,25 @@
 <robot name="navigator" xmlns:xacro="http://ros.org/wiki/xacro">
   <!-- Defines the base vehicle -->
-  <xacro:include filename="$(find wamv_description)/urdf/wamv_base.urdf.xacro" />
+  <xacro:include filename="$(find wamv_description)/urdf/wamv_base.urdf.xacro"/>
   <!-- Fixed frames for sensors -->
-  <xacro:include filename="$(find navigator_gazebo)/urdf/fixed_link.xacro" />
-  <xacro:include filename="$(find navigator_gazebo)/urdf/sylphase.xacro" />
-  <xacro:fixed_link name="measurement"
-                    xyz="1.2319 0 1.2" rpy="0 0 0" />
-  <xacro:sylphase name="ins"
-                  xyz="0.579628 0.136525 1.392278" rpy="0 0 0" />
-  <xacro:fixed_link name="velodyne" parent="measurement"
-                    xyz="-0.277622 0 0.648208" rpy="0 0 0" />
-  <xacro:fixed_link name="sick" parent="measurement"
-                    xyz="0.5334 -0.0254 -0.6858" rpy="0 0 0" />
-  <xacro:fixed_link name="pinger_direction" parent="velodyne"
-                    xyz="0.8382 0 -2.0828" rpy="0 0 0" />
+  <xacro:include filename="$(find navigator_gazebo)/urdf/fixed_link.xacro"/>
+  <xacro:include filename="$(find navigator_gazebo)/urdf/sylphase.xacro"/>
+  <xacro:fixed_link name="measurement" xyz="1.2319 0 1.2" rpy="0 0 0"/>
+  <xacro:sylphase name="ins" xyz="0.579628 0.136525 1.392278" rpy="0 0 0"/>
+  <xacro:fixed_link name="velodyne" parent="measurement" xyz="-0.277622 0 0.648208" rpy="0 0 0"/>
+  <xacro:fixed_link name="sick" parent="measurement" xyz="0.5334 -0.0254 -0.6858" rpy="0 0 0"/>
+  <xacro:fixed_link name="pinger_direction" parent="velodyne" xyz="0.8382 0 -2.0828" rpy="0 0 0"/>
   <!-- Camera frames with gazebo simulation plugins -->
-  <xacro:include filename="$(find navigator_gazebo)/urdf/camera.xacro" />
-  <xacro:navigator_camera name="front_left_cam" parent="velodyne"
-                          namespace="/camera/front/left"
-                          xyz="0.294 0.1 -0.45"
-                          rpy="0 0.258 0" />
-  <xacro:navigator_camera name="front_right_cam" parent="velodyne"
-                           namespace="/camera/front/right"
-                          xyz="0.294 -0.099 -0.45"
-                          rpy="0 0.258 0" />
-  <xacro:navigator_camera name="starboard_cam" parent="measurement"
-                          namespace="/camera/starboard"
-                          xyz="-0.4191 -0.6985 0.2159"
-                          rpy="0 0 -1.570796" />
-  <xacro:fixed_link name="shooter" parent="starboard_cam" xyz="0 0 0.2" rpy="0 0 0" />
+  <xacro:include filename="$(find navigator_gazebo)/urdf/camera.xacro"/>
+  <xacro:navigator_camera name="front_left_cam" parent="velodyne" namespace="/camera/front/left" xyz="0.294 0.1 -0.45" rpy="0 0.258 0"/>
+  <xacro:navigator_camera name="front_right_cam" parent="velodyne" namespace="/camera/front/right" xyz="0.294 -0.099 -0.45" rpy="0 0.258 0"/>
+  <xacro:navigator_camera name="starboard_cam" parent="measurement" namespace="/camera/starboard" xyz="-0.4191 -0.6985 0.2159" rpy="0 0 -1.570796"/>
+  <xacro:fixed_link name="shooter" parent="starboard_cam" xyz="0 0 0.2" rpy="0 0 0"/>
   <!-- Add 4 thrusters -->
-  <xacro:include filename="$(find navigator_gazebo)/urdf/thruster.xacro" />
-  <xacro:navigator_thruster name="BL" x="-1.9304" y="1.016"   yaw="0.785398" />
-  <xacro:navigator_thruster name="BR" x="-1.9304" y="-1.016"  yaw="-0.785398" />
-  <xacro:navigator_thruster name="FL" x="1.5748"  y="0.6096"  yaw="-0.785398" />
-  <xacro:navigator_thruster name="FR" x="1.5748"  y="-0.6096" yaw="0.785398" />
+  <xacro:include filename="$(find navigator_gazebo)/urdf/thruster.xacro"/>
+  <xacro:navigator_thruster name="BL" x="-1.9304" y="1.016" yaw="0.785398"/>
+  <xacro:navigator_thruster name="BR" x="-1.9304" y="-1.016" yaw="-0.785398"/>
+  <xacro:navigator_thruster name="FL" x="1.5748" y="0.6096" yaw="-0.785398"/>
+  <xacro:navigator_thruster name="FR" x="1.5748" y="-0.6096" yaw="0.785398"/>
   <!-- Plugin to imitate roboteq motor driver for thrusters -->
   <gazebo>
@@ -52,8 +38,7 @@
     </plugin>
   </gazebo>
-  <xacro:fixed_link name="hydrophones" parent="base_link"
-                    xyz="0.102 -.635 -0.324" rpy="0 0 0" />
+  <xacro:fixed_link name="hydrophones" parent="base_link" xyz="0.102 -.635 -0.324" rpy="0 0 0"/>
   <!-- Attach hydrodynamics plugin -->
-  <xacro:include filename="$(find wamv_gazebo)/urdf/macros.xacro" />
+  <xacro:include filename="$(find wamv_gazebo)/urdf/macros.xacro"/>
   <xacro:usv_dynamics_gazebo name="wamv_dynamics_plugin"/>
   <!-- Attach wind plugin -->

File: NaviGator/simulation/navigator_gazebo/urdf/sylphase.xacro (robot description, xacro)
@@ -1,18 +1,16 @@
 <?xml version="1.0"?>
 <robot xmlns:xacro="http://ros.org/wiki/xacro">
-  <xacro:macro  name="sylphase"
-                params="name='ins'
+  <xacro:macro name="sylphase" params="name='ins'
                         xyz:='0 0 0' rpy:='0 0 0'">
-    <xacro:include filename="$(find navigator_gazebo)/urdf/fixed_link_persistent.xacro" />
-    <link name="${name}">
-    </link>
+    <xacro:include filename="$(find navigator_gazebo)/urdf/fixed_link_persistent.xacro"/>
+    <link name="${name}"/>
     <gazebo reference="${name}">
-      <sensor name="${name}_imu" type="imu" />
-      <sensor name="${name}_gps" type="gps" />
+      <sensor name="${name}_imu" type="imu"/>
+      <sensor name="${name}_gps" type="gps"/>
     </gazebo>
     <joint name="${name}_to_base_link" type="fixed">
-      <parent link="base_link" />
-      <child link="${name}" />
-      <origin xyz="${xyz}" rpy="${rpy}" />
+      <parent link="base_link"/>
+      <child link="${name}"/>
+      <origin xyz="${xyz}" rpy="${rpy}"/>
     </joint>
     <gazebo>

File: NaviGator/simulation/navigator_gazebo/urdf/thruster.xacro (robot description, xacro)
@@ -2,12 +2,12 @@
 <robot xmlns:xacro="http://ros.org/wiki/xacro" name="wam-v-two-engines">
   <!-- Macro for inserting an engine with its propeller. -->
-  <xacro:macro  name="navigator_thruster" params="name x y yaw">
+  <xacro:macro name="navigator_thruster" params="name x y yaw">
     <!-- Location of propeller from origin of engine -->
-    <xacro:property name="prop_x_offset" value="-0.278156" />
+    <xacro:property name="prop_x_offset" value="-0.278156"/>
     <!-- Transform engine position so macro position is position of propeller -->
-    <xacro:property name="s_yaw" value="${sin(yaw)}" />
-    <xacro:property name="c_yaw" value="${cos(yaw)}" />
-    <xacro:property name="x_engine" value="${x + c_yaw*(-prop_x_offset) - s_yaw*(0)} " />
-    <xacro:property name="y_engine" value="${y + s_yaw*(-prop_x_offset) + c_yaw*(0)} " />
+    <xacro:property name="s_yaw" value="${sin(yaw)}"/>
+    <xacro:property name="c_yaw" value="${cos(yaw)}"/>
+    <xacro:property name="x_engine" value="${x + c_yaw*(-prop_x_offset) - s_yaw*(0)} "/>
+    <xacro:property name="y_engine" value="${y + s_yaw*(-prop_x_offset) + c_yaw*(0)} "/>
     <link name="${name}_engine_link">
       <visual>
@@ -17,13 +17,13 @@
       </visual>
       <collision name="${name}_engine_vertical_axis_collision">
-        <origin xyz="-0.16 0 -0.24" rpy="0 0 0" />
+        <origin xyz="-0.16 0 -0.24" rpy="0 0 0"/>
         <geometry>
-          <box size="0.2 0.15 0.83" />
+          <box size="0.2 0.15 0.83"/>
         </geometry>
       </collision>
       <collision name="${name}_engine_rear_end_collision">
-        <origin xyz="-0.34 0 0.12" rpy="0 0 0" />
+        <origin xyz="-0.34 0 0.12" rpy="0 0 0"/>
         <geometry>
-          <box size="0.12 0.15 0.12" />
+          <box size="0.12 0.15 0.12"/>
         </geometry>
       </collision>
@@ -40,7 +40,7 @@
       </visual>
       <collision name="${name}_propeller_collision">
-        <origin xyz="-0.08 0 0" rpy="0 1.57 0" />
+        <origin xyz="-0.08 0 0" rpy="0 1.57 0"/>
         <geometry>
-          <cylinder length="0.18" radius="0.24" />
+          <cylinder length="0.18" radius="0.24"/>
         </geometry>
       </collision>
@@ -60,6 +60,6 @@
       <child link="${name}_propeller_link"/>
       <origin rpy="0 0 0" xyz="${prop_x_offset} 0 -0.509371"/>
-      <limit effort="400" velocity="100" />
-      <dynamics friction="100" damping="0.3" />
+      <limit effort="400" velocity="100"/>
+      <dynamics friction="100" damping="0.3"/>
     </joint>
     <transmission name="${name}_thruster_transmission">

File: NaviGator/simulation/navigator_gazebo/worlds/course.world.xacro (robot description, xacro)
@@ -1,3 +1,3 @@
-<?xml version="1.0" ?>
+<?xml version="1.0"?>
 <!-- World containing sandisland model and some course challenges -->
 <sdf version="1.6" xmlns:xacro="http://ros.org/wiki/xacro">
@@ -11,6 +11,6 @@
       <max_step_size>0.01</max_step_size>
     </physics>
-    <xacro:include filename="$(find vrx_gazebo)/worlds/xacros/sandisland_minus_scene.xacro" />
-    <xacro:sandisland_minus_scene />
+    <xacro:include filename="$(find vrx_gazebo)/worlds/xacros/sandisland_minus_scene.xacro"/>
+    <xacro:sandisland_minus_scene/>
     <include>
       <uri>model://robotx_navigation_challenge</uri>
@@ -38,13 +38,13 @@
     <include>
       <uri>model://ring_recovery_reference_buoy</uri>
-      <pose>65 20 0 0 0 0 </pose>
+      <pose>65 20 0 0 0 0</pose>
     </include>
     <!-- Find totems challenge -->
     <include>
       <uri>model://find_totems_challenge</uri>
-      <pose>35 50 0 0 0 0 </pose>
+      <pose>35 50 0 0 0 0</pose>
     </include>
     <!-- Run simulated PCODAR -->
-    <plugin name="pcodar_gazebo" filename="libpcodar_gazebo.so" />
+    <plugin name="pcodar_gazebo" filename="libpcodar_gazebo.so"/>
   </world>
 </sdf>
