Commit message: Added changes from recent testings - Changed the thruster ID values to correspond to the current thruster   connection setup. - Changed FRV thruster direction from -1Z to +1Z. - Changed PID values for the sub. Values are still not ideal and will be   adjusted over the next few testing sessions. - Changed the identifier for the USB to CAN board's USB to serial   converter. - Changed tcp address for the depth sensor, imu, and dvl connection   scripts to their ip addresses instead of their DNS names (there is an issue with the DNS server in the network box, or in the lab, or both). - Made changes to the sub8.urdf.xacro for gazebo to avoid URDF inertia   warning. - Added bag_debugging_controller.launch file which is a launch file to   record bags for debugging the PID controller on the sub.

File: SubjuGator/simulation/subjugator_gazebo/urdf/sub8.urdf.xacro (robot description, xacro)
@@ -11,5 +11,12 @@
   <xacro:include filename="$(find mil_gazebo)/xacro/passive_sonar.xacro"/>
   <xacro:include filename="$(find mil_gazebo)/xacro/inclinometer.xacro"/>
+  <!-- dummy link and joint to avoid URDF inertia warning-->
+  <link name="dummy"/>
   <!-- Base link of sub -->
+  <joint name="dummy_joint" type="fixed">
+    <parent link="dummy"/>
+    <child link="base_link"/>
+  </joint>
+  <!-- base link -->
   <link name="base_link">
     <inertial>

Commit message: Modify URDF fix to fix /mission_server crash - Another URDF xacro fix has been applied to the URDF xacro file using these ROS forum posts as reference: https://answers.ros.org/question/393006/urdf-link-not-properly-fixed-to-world/, https://answers.ros.org/question/192817/error-msg-the-root-link_base-has-an-inertia-specified-in-the-urdf-but-kdl/. NOTE: This is not a complete fix yet. I'm getting a tf republisher error that 'base_link' and 'map' do not have a connection with TF having 2+ unconnected trees. Additionally, gazebogui does not work since the /gzclient/set_physics_properties service is not advertised (even though /gazebo/set_physics_properties is).

File: SubjuGator/simulation/subjugator_gazebo/urdf/sub8.urdf.xacro (robot description, xacro)
@@ -11,12 +11,6 @@
   <xacro:include filename="$(find mil_gazebo)/xacro/passive_sonar.xacro"/>
   <xacro:include filename="$(find mil_gazebo)/xacro/inclinometer.xacro"/>
-  <!-- dummy link and joint to avoid URDF inertia warning-->
-  <link name="dummy"/>
+  <link name="world"/>
   <!-- Base link of sub -->
-  <joint name="dummy_joint" type="fixed">
-    <parent link="dummy"/>
-    <child link="base_link"/>
-  </joint>
-  <!-- base link -->
   <link name="base_link">
     <inertial>
@@ -37,4 +31,8 @@
     </collision>
   </link>
+  <joint name="dummy_joint" type="fixed">
+    <parent link="world"/>
+    <child link="base_link"/>
+  </joint>
   <!-- Sensors -->
   <xacro:mil_fixed_link name="front_stereo" parent="base_link" xyz="0.2559 0 0.1707" rpy="0 0 0"/>

Commit message: Testing changes (#1062)
* Added changes from recent testings
- Changed the thruster ID values to correspond to the current thruster
  connection setup.
- Changed FRV thruster direction from -1Z to +1Z.
- Changed PID values for the sub. Values are still not ideal and will be
  adjusted over the next few testing sessions.
- Changed the identifier for the USB to CAN board's USB to serial
  converter.
- Changed tcp address for the depth sensor, imu, and dvl connection
  scripts to their ip addresses instead of their DNS names (there is an
issue with the DNS server in the network box, or in the lab, or both).
- Made changes to the sub8.urdf.xacro for gazebo to avoid URDF inertia
  warning.
- Added bag_debugging_controller.launch file which is a launch file to
  record bags for debugging the PID controller on the sub.

* Add documentation for bag_debugging_controller.launch

* pre-commit and CI fixes...probably

* Added documentation about PID controller
- Added documentation page about PID controller containing information
about the bag_debugging_controller.launch file and some tips for how to
tune the PID controller.
- Reverted subjugator_launch/readme.md changes to reflect moving to a
new documentation page.
- Modified adaptive controller values to remove commented out kd values.

* Modify URDF fix to fix /mission_server crash
- Another URDF xacro fix has been applied to the URDF xacro file using
these ROS forum posts as reference:
https://answers.ros.org/question/393006/urdf-link-not-properly-fixed-to-world/,
https://answers.ros.org/question/192817/error-msg-the-root-link_base-has-an-inertia-specified-in-the-urdf-but-kdl/.
NOTE: This is not a complete fix yet. I'm getting a tf republisher error
that 'base_link' and 'map' do not have a connection with TF having 2+
unconnected trees. Additionally, gazebogui does not work since
the /gzclient/set_physics_properties service is not advertised (even
though /gazebo/set_physics_properties is).

* Add support for simulation vs physical PID gains

---------

Co-authored-by: Cameron Brown <me@cbrxyz.com>
Co-authored-by: cameron brown <52760912+cbrxyz@users.noreply.github.com>

File: SubjuGator/simulation/subjugator_gazebo/urdf/sub8.urdf.xacro (robot description, xacro)
@@ -11,4 +11,5 @@
   <xacro:include filename="$(find mil_gazebo)/xacro/passive_sonar.xacro"/>
   <xacro:include filename="$(find mil_gazebo)/xacro/inclinometer.xacro"/>
+  <link name="world"/>
   <!-- Base link of sub -->
   <link name="base_link">
@@ -30,4 +31,8 @@
     </collision>
   </link>
+  <joint name="dummy_joint" type="fixed">
+    <parent link="world"/>
+    <child link="base_link"/>
+  </joint>
   <!-- Sensors -->
   <xacro:mil_fixed_link name="front_stereo" parent="base_link" xyz="0.2559 0 0.1707" rpy="0 0 0"/>

Commit message: Limit TF_REPEATED_DATA messages by checking for repeated transforms, also remove dummy world join to rejoin map + base_link trees in simulation

File: SubjuGator/simulation/subjugator_gazebo/urdf/sub8.urdf.xacro (robot description, xacro)
@@ -11,5 +11,4 @@
   <xacro:include filename="$(find mil_gazebo)/xacro/passive_sonar.xacro"/>
   <xacro:include filename="$(find mil_gazebo)/xacro/inclinometer.xacro"/>
-  <link name="world"/>
   <!-- Base link of sub -->
   <link name="base_link">
@@ -31,8 +30,4 @@
     </collision>
   </link>
-  <joint name="dummy_joint" type="fixed">
-    <parent link="world"/>
-    <child link="base_link"/>
-  </joint>
   <!-- Sensors -->
   <xacro:mil_fixed_link name="front_stereo" parent="base_link" xyz="0.2559 0 0.1707" rpy="0 0 0"/>
